Commit message: Get real robot working
done to minute 24 th of vid 2 ros2_control

    modified:   config/my_controllers.yaml

    modified:   description/ros2_control.xacro

    new file:   launch/launch_robot.launch.py

	new file:   launch/rplidar.launch.py

	modified:   launch/rsp.launch.py

Chinh sua file /home/pi/realduopi1_ws/src/diffdrive_arduino/hardware/include/diffdrive_arduino/arduino_comms.hpp

    Them ham send_msg_only va thay the no trong ham con cua ham set_motor_values

    Doi cho val_1 val_2 vi encoder bi nguoc

File: description/ros2_control.xacro (robot description, xacro)
@@ -1,5 +1,34 @@
 <?xml version="1.0"?> <!-- Vid 2 SECOND STEP -->
 <robot xmlns:xacro="http://www.ros.org/wiki/xacro">
-    <ros2_control name="GazeboSystem" type="system">
+    <ros2_control name="Realrobot" type="system">
+        <hardware>
+            <plugin>diffdrive_arduino/DiffDriveArduinoHardware</plugin> <!-- as -->
+            <param name="left_wheel_name">left_wheel_joint</param>
+            <param name="right_wheel_name">right_wheel_joint</param>
+            <param name="loop_rate">30</param>
+            <!-- <param name="device">/dev/ttuUSB0</param>  -->  <!-- thay sau /dev/ bang duong dan by-path-->
+            <param name="device">/dev/serial/by-path/platform-fd500000.pcie-pci-0000:01:00.0-usb-0:1.4:1.0-port0</param>
+            <param name="baud_rate">115200</param>
+            <param name="timeout_ms">1000</param> <!-- thay timout bang timeout_ms -->
+            <param name="enc_counts_per_rev">3960</param>
+        </hardware>
+        <joint name="right_wheel_joint">
+            <command_interface name="velocity">
+                <param name="min">-10</param>
+                <param name="max">10</param>
+            </command_interface>
+            <state_interface name="position"/> <!-- position dung truoc velocity moi duoc -->
+            <state_interface name="velocity"/>
+        </joint>
+        <joint name="left_wheel_joint">
+            <command_interface name="velocity">
+                <param name="min">-10</param>
+                <param name="max">10</param>
+            </command_interface>
+            <state_interface name="position"/> <!-- position dung truoc velocity moi duoc -->
+            <state_interface name="velocity"/>
+        </joint>
+    </ros2_control>
+    <!-- <ros2_control name="GazeboSystem" type="system">
         <hardware>
             <plugin>gazebo_ros2_control/GazeboSystem</plugin>
@@ -21,5 +50,5 @@
             <state_interface name="position"/>
         </joint>
-    </ros2_control>
+    </ros2_control> -->
     <gazebo>
         <plugin name="gazebo_ros2_control" filename="libgazebo_ros2_control.so">
